File: sources/bridgeconnector/nexys3-spartan3-starter/vhdci-fx2.brd (EAGLE design)
At the start: 44.1 x 76.2 mm, 7 parts, among them X1 BU-SMA-V

Commit message: bla
Routing:
- net GND: track 0.00 -> 17.9 mm
Changed lines of the file:
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@@
 <setting verticaltext="up"/>
 </settings>
-<grid distance="0.025" unitdist="inch" unit="inch" style="lines" multiple="1" display="yes" altdistance="0.025" altunitdist="inch" altunit="inch"/>
+<grid distance="0.0125" unitdist="inch" unit="inch" style="lines" multiple="1" display="yes" altdistance="0.025" altunitdist="inch" altunit="inch"/>
 <layers>
 <layer number="1" name="Top" color="4" fill="1" visible="yes" active="yes"/>
@@
 <contactref element="U$2" pad="V39"/>
 <contactref element="U$2" pad="V36"/>
+<wire x1="13.6" y1="28" x2="15.2" y2="28" width="0.3048" layer="1"/>
+<wire x1="15.2" y1="28" x2="16" y2="28.8" width="0.3048" layer="1"/>
+<wire x1="16" y1="28.8" x2="16.8" y2="28.8" width="0.3048" layer="1"/>
+<wire x1="16.8" y1="28.8" x2="18.005" y2="28.8" width="0.4064" layer="1"/>
+<wire x1="18.005" y1="28.8" x2="19.05" y2="29.845" width="0.4064" layer="1"/>
+<wire x1="19.05" y1="29.845" x2="29.845" y2="29.845" width="0.4064" layer="1"/>
+<wire x1="29.845" y1="29.845" x2="30.48" y2="30.48" width="0.4064" layer="1"/>
 <wire x1="48.26" y1="62.23" x2="48.26" y2="64.77" width="0" layer="19" extent="1-1"/>
 <wire x1="46.355" y1="60.96" x2="48.26" y2="62.23" width="0" layer="19" extent="1-1"/>
@@
 <wire x1="33.02" y1="30.48" x2="33.02" y2="43.18" width="0" layer="19" extent="1-1"/>
 <wire x1="30.48" y1="30.48" x2="33.02" y2="30.48" width="0" layer="19" extent="1-1"/>
-<wire x1="33.02" y1="17.78" x2="33.02" y2="30.48" width="0" layer="19" extent="1-1"/>
-<wire x1="30.48" y1="17.78" x2="33.02" y2="17.78" width="0" layer="19" extent="1-1"/>
-<wire x1="30.48" y1="5.08" x2="30.48" y2="17.78" width="0" layer="19" extent="1-1"/>
-<wire x1="24.1399" y1="68.5701" x2="30.48" y2="55.88" width="0" layer="19" extent="1-1"/>
-<wire x1="24.1399" y1="73.6699" x2="24.1399" y2="68.5701" width="0" layer="19" extent="1-1"/>
-<wire x1="19.0401" y1="73.6699" x2="24.1399" y2="73.6699" width="0" layer="19" extent="1-1"/>
-<wire x1="19.0401" y1="68.5701" x2="24.1399" y2="68.5701" width="0" layer="19" extent="1-1"/>
-<wire x1="14.75" y1="43.2" x2="30.48" y2="43.18" width="0" layer="19" extent="1-1"/>
-<wire x1="12.4" y1="42.8" x2="14.75" y2="43.2" width="0" layer="19" extent="1-1"/>
-<wire x1="13.6" y1="40.8" x2="12.4" y2="42.8" width="0" layer="19" extent="1-1"/>
-<wire x1="11.25" y1="40.4" x2="13.6" y2="40.8" width="0" layer="19" extent="1-1"/>
-<wire x1="14.75" y1="38.4" x2="13.6" y2="40.8" width="0" layer="19" extent="1-1"/>
-<wire x1="12.4" y1="38" x2="14.75" y2="38.4" width="0" layer="19" extent="1-1"/>
-<wire x1="13.6" y1="36" x2="12.4" y2="38" width="0" layer="19" extent="1-1"/>
-<wire x1="11.25" y1="35.6" x2="13.6" y2="36" width="0" layer="19" extent="1-1"/>
-<wire x1="13.6" y1="28" x2="11.25" y2="35.6" width="0" layer="19" extent="1-1"/>
 <wire x1="11.25" y1="27.6" x2="13.6" y2="28" width="0" layer="19" extent="1-1"/>
-<wire x1="14.75" y1="25.6" x2="13.6" y2="28" width="0" layer="19" extent="1-1"/>
+<wire x1="14.75" y1="25.6" x2="15.2" y2="28" width="0" layer="19" extent="1-1"/>
 <wire x1="12.4" y1="25.2" x2="14.75" y2="25.6" width="0" layer="19" extent="1-1"/>
 <wire x1="13.6" y1="23.2" x2="12.4" y2="25.2" width="0" layer="19" extent="1-1"/>
@@
 <wire x1="14.75" y1="20.8" x2="12.3" y2="20.4" width="0" layer="19" extent="1-1"/>
 <wire x1="11.15" y1="18" x2="13.6" y2="18.4" width="0" layer="19" extent="1-1"/>
+<wire x1="13.6" y1="36" x2="16" y2="28.8" width="0" layer="19" extent="1-1"/>
+<wire x1="12.4" y1="38" x2="13.6" y2="36" width="0" layer="19" extent="1-1"/>
+<wire x1="14.75" y1="38.4" x2="12.4" y2="38" width="0" layer="19" extent="1-1"/>
+<wire x1="11.25" y1="35.6" x2="13.6" y2="36" width="0" layer="19" extent="1-1"/>
+<wire x1="13.6" y1="40.8" x2="14.75" y2="38.4" width="0" layer="19" extent="1-1"/>
+<wire x1="12.4" y1="42.8" x2="13.6" y2="40.8" width="0" layer="19" extent="1-1"/>
+<wire x1="14.75" y1="43.2" x2="12.4" y2="42.8" width="0" layer="19" extent="1-1"/>
+<wire x1="11.25" y1="40.4" x2="13.6" y2="40.8" width="0" layer="19" extent="1-1"/>
+<wire x1="30.48" y1="17.78" x2="29.845" y2="29.845" width="0" layer="19" extent="1-1"/>
+<wire x1="33.02" y1="17.78" x2="30.48" y2="17.78" width="0" layer="19" extent="1-1"/>
+<wire x1="30.48" y1="5.08" x2="30.48" y2="17.78" width="0" layer="19" extent="1-1"/>
+<wire x1="24.1399" y1="68.5701" x2="30.48" y2="55.88" width="0" layer="19" extent="1-1"/>
+<wire x1="24.1399" y1="73.6699" x2="24.1399" y2="68.5701" width="0" layer="19" extent="1-1"/>
+<wire x1="19.0401" y1="73.6699" x2="24.1399" y2="73.6699" width="0" layer="19" extent="1-1"/>
+<wire x1="19.0401" y1="68.5701" x2="24.1399" y2="68.5701" width="0" layer="19" extent="1-1"/>
 </signal>
 <signal name="VCC5V">
@@
 <wire x1="16.8" y1="16" x2="17.27" y2="16" width="0.4064" layer="1"/>
 <wire x1="17.27" y1="16" x2="20.32" y2="19.05" width="0.4064" layer="1"/>
-<wire x1="20.32" y1="19.05" x2="20.32" y2="29.21" width="0.4064" layer="1"/>
-<via x="20.32" y="29.21" extent="1-16" drill="0.5"/>
-<wire x1="20.32" y1="29.21" x2="20.32" y2="30.48" width="0.4064" layer="16"/>
-<via x="20.32" y="30.48" extent="1-16" drill="0.5"/>
-<wire x1="20.32" y1="30.48" x2="20.32" y2="52.705" width="0.4064" layer="1"/>
+<wire x1="20.32" y1="19.05" x2="20.32" y2="28.8925" width="0.4064" layer="1"/>
+<via x="20.32" y="28.8925" extent="1-16" drill="0.5"/>
+<wire x1="20.32" y1="28.8925" x2="20.32" y2="30.7975" width="0.4064" layer="16"/>
+<via x="20.32" y="30.7975" extent="1-16" drill="0.5"/>
+<wire x1="20.32" y1="30.7975" x2="20.32" y2="52.705" width="0.4064" layer="1"/>
 <wire x1="20.32" y1="52.705" x2="28.575" y2="60.96" width="0.4064" layer="16"/>
 <wire x1="28.575" y1="60.96" x2="30.48" y2="60.96" width="0.4064" layer="16"/>
@@
 <wire x1="17.145" y1="14.605" x2="17.78" y2="14.605" width="0.4064" layer="1"/>
 <wire x1="17.78" y1="14.605" x2="21.59" y2="18.415" width="0.4064" layer="1"/>
-<wire x1="21.59" y1="18.415" x2="21.59" y2="29.21" width="0.4064" layer="1"/>
-<via x="21.59" y="29.21" extent="1-16" drill="0.5"/>
-<wire x1="21.59" y1="29.21" x2="21.59" y2="30.48" width="0.4064" layer="16"/>
-<via x="21.59" y="30.48" extent="1-16" drill="0.5"/>
-<wire x1="21.59" y1="30.48" x2="21.59" y2="51.435" width="0.4064" layer="1"/>
+<wire x1="21.59" y1="18.415" x2="21.59" y2="28.8925" width="0.4064" layer="1"/>
+<via x="21.59" y="28.8925" extent="1-16" drill="0.5"/>
+<wire x1="21.59" y1="28.8925" x2="21.59" y2="30.7975" width="0.4064" layer="16"/>
+<via x="21.59" y="30.7975" extent="1-16" drill="0.5"/>
+<wire x1="21.59" y1="30.7975" x2="21.59" y2="51.435" width="0.4064" layer="1"/>
 <wire x1="21.59" y1="51.435" x2="28.575" y2="58.42" width="0.4064" layer="16"/>
 <wire x1="28.575" y1="58.42" x2="30.48" y2="58.42" width="0.4064" layer="16"/>
