File: sources/bridgeconnector/nexys3-spartan3-starter/vhdci-fx2.sch (EAGLE design)
At the start: 7 parts, among them X1 BU-SMA-V

Commit message: bla
Changed lines of the file:
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@@
 <wire x1="124.46" y1="43.18" x2="114.3" y2="43.18" width="0.1524" layer="91"/>
 <pinref part="U$1" gate="HIROSE100" pin="IO16"/>
+<label x="116.84" y="43.18" size="1.778" layer="95"/>
 </segment>
 <segment>
@@
 <wire x1="124.46" y1="45.72" x2="114.3" y2="45.72" width="0.1524" layer="91"/>
 <pinref part="U$1" gate="HIROSE100" pin="IO17"/>
+<label x="116.84" y="45.72" size="1.778" layer="95"/>
 </segment>
 <segment>
@@
 <wire x1="124.46" y1="83.82" x2="114.3" y2="83.82" width="0.1524" layer="91"/>
 <pinref part="U$1" gate="HIROSE100" pin="IO32"/>
-</segment>
-<segment>
+<label x="114.3" y="83.82" size="1.778" layer="95"/>
+</segment>
+<segment>
