File: sources/bridgeconnector/nexys3-spartan3-starter/vhdci-fx2-gnd.brd (EAGLE design)
At the start: 44.1 x 76.2 mm, 9 parts, among them X1 CLK, X2 TRIGGER

Commit message: board layout
Parts:
- moved X2 1.27 mm to (11.4, 70.5)
Routing:
- net CLKIN_D: track 23.0 -> 73.9 mm, vias 0 -> 2
- net DOUT12: track 0.00 -> 43.6 mm, vias 0 -> 1
- net DOUT14: track 0.00 -> 43.2 mm, vias 0 -> 1
- net DOUT10: track 0.00 -> 43.2 mm, vias 0 -> 1
- net DOUT8: track 0.00 -> 41.6 mm, vias 0 -> 1
- net DOUT13: track 0.00 -> 39.6 mm
- net DOUT15: track 0.00 -> 39.3 mm
- net DIN8: track 0.00 -> 39.3 mm, vias 0 -> 1
- net DOUT11: track 0.00 -> 39.2 mm
- net DIN14: track 0.00 -> 39.1 mm, vias 0 -> 1
- net DIN9: track 0.00 -> 39.0 mm
- net DIN15: track 0.00 -> 39.0 mm
- net DOUT4: track 0.00 -> 38.3 mm, vias 0 -> 1
- net DOUT2: track 0.00 -> 38.0 mm, vias 0 -> 1
- net DOUT6: track 0.00 -> 37.5 mm
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- added copper zone on layer 1, net GND
- added copper zone on layer 16, net GND

Commit message: bla
Other:
- board text added: "/home/jkaps/public_html/cerg/design/CERG-logo-with-url-bw.bmp"
- board text added: "1"
- board text added: "2"
- board text added: "49"
- board text added: "50"
- board text added: "A"
- board text added: "Alternate DUT"
- board text added: "B"
- board text added: "CLK"
- board text added: "CLK_C2D"
- board text added: "CLK_E2C"
- board text added: "CLK_E2D"
- board text added: "Control"
- board text added: "DUT"
- board text added: "JP1"
- board text added: "JP2"
- board text added: "JP3"
- board text added: "JP4"
- board text added: "JP5"
- board text added: "TRIGGER"
- board text added: "TRIGGER_2D"
- board text added: "X1"
- board text added: "X2"

Commit message: bla
Connections:
- net RST: now also U$2.V49; no longer U$2.V54
- net TRIGGER: now also U$2.V54; no longer U$2.V49
Routing:
- net TRIGGER: track 52.4 -> 56.6 mm
- net RST: track 51.1 -> 49.4 mm, vias 2 -> 3
- net CLKIN_C: vias 1 -> 0
Other:
- board text added: "FOBOS VHDCI to FX2 Bridge Connector"
- board text added: "cryptography.gmu.edu"
- board text added: "rev 1.0"

Commit message: clk_d2e
Parts:
- removed JP2: CLK_E2D, jumper:JP1
- added JP7: CLK_E2D, jumper:JP2Q
Connections:
- new net CLKOUT_D: DUT.A47, JP7.4
- net CLKIN_D: now also JP7.2; no longer JP2.2
- net N$3: now also JP7.1, JP7.3; no longer JP2.1
Routing:
- net CLKOUT_D: track 0.00 -> 8.08 mm
- net CLKIN_D: track 73.9 -> 77.3 mm, vias 2 -> 1
- net N$3: track 32.9 -> 33.8 mm
Other:
- board text added: "D2E"
- board text added: "E2D"
- board text added: "rev 1.1"
- board text removed: "CLK_E2D"
- board text removed: "rev 1.0"
