File: hardware/fobos-dut/dut-artix7-a12t/fpga.sch (KiCad schematic (older format))
At the start: 28 parts

Commit message: started adding FPGA to Artix7 DUT
Parts:
- removed C? (x3): 100nF, Capacitor_SMD:C_0603_1608Metric, symbol Device:C
- removed J?: Target, Connector_IDC:IDC-Header_2x10_P2.54mm_Horizontal, symbol Connector_Generic:Conn_02x10_Odd_Even
- removed J?: Pmod 2x6, symbol Connector_Generic:Conn_02x06_Top_Bottom
- removed R? (x12): 22R, Resistor_SMD:R_0603_1608Metric, symbol Device:R
- removed R? (x8): 200R, Resistor_SMD:R_0603_1608Metric, symbol Device:R
- removed U? (x3): SP3003-04ATG, Package_SO:MSOP-10_3x3mm_P0.5mm, symbol cerg:SP3003-04ATG
- added C?: 100n, Capacitor_SMD:C_0603_1608Metric, symbol Device:C
- added R? (x3): 33R, Resistor_SMD:R_0603_1608Metric, symbol Device:R
- added R?: 4K7, Resistor_SMD:R_0603_1608Metric, symbol Device:R
- added R? (x2): 1R, Resistor_SMD:R_0603_1608Metric, symbol Device:R
- added U1: XC7A12T-CSG325, Package_BGA:Xilinx_CSG325, symbol cerg:XC7A12T-CSG325
- added U?: W25Q32JVSS, Package_SO:SOIC-8_5.23x5.23mm_P1.27mm, symbol Memory_Flash:W25Q32JVSS
Connections:
- net labels added: FPGA_CCLK, HOLD, VCCIO, WP
- net labels removed: +3V3, Aux, CLK_C2D, CLK_D2C, CV_RST, CW_HS1, CW_HS2, CW_MISO, CW_MOSI, CW_PDIC, CW_PDID, CW_SCK, CW_TARG1, CW_TARG2, CW_TARG3, CW_TARG4, CW_VREF, DIO0, DIO1, DIO2, DIO3, FS_3V3, FS_5V, IO, RST, Ready, TF, Valid
- wire segments 139 -> 39
Other:
- note added: "JA can be \ndifferentially\nrouted"
- note removed: "ESD Protection"
- note removed: "FOBOS Target Connector"
- note removed: "PMOD Connector"

Commit message: artix 7 dut PCB work
Other:
- moved on the sheet: U1C
Changed lines of the file:
@@
 L cerg:XC7A12T-CSG325 U1
 U 3 1 5F268106
-P 8800 2550
-F 0 "U1" H 8800 1175 50  0000 C CNN
-F 1 "XC7A12T-CSG325" H 8800 1084 50  0000 C CNN
-F 2 "Package_BGA:Xilinx_CSG325" H 8800 2550 50  0001 C CNN
-F 3 "https://www.xilinx.com/support/documentation/data_sheets/ds180_7Series_Overview.pdf" H 8800 2550 50  0001 C CNN
-	3    8800 2550
+P 8650 3000
+F 0 "U1" H 8650 1625 50  0000 C CNN
+F 1 "XC7A12T-CSG325" H 8650 1534 50  0000 C CNN
+F 2 "Package_BGA:Xilinx_CSG325" H 8650 3000 50  0001 C CNN
+F 3 "https://www.xilinx.com/support/documentation/data_sheets/ds180_7Series_Overview.pdf" H 8650 3000 50  0001 C CNN
+	3    8650 3000
 	1    0    0    -1
 $EndComp

Commit message: artix 7 dut updates
Parts:
- gave numbers to parts that had none: 8
Changed lines of the file:
@@
 JA can be \ndifferentially\nrouted
 $Comp
-L Memory_Flash:W25Q32JVSS U?
+L Memory_Flash:W25Q32JVSS U7
 U 1 1 5F5D51AE
 P 1700 2100
-F 0 "U?" H 1700 2681 50  0000 C CNN
-F 1 "W25Q32JVSS" H 1700 2590 50  0000 C CNN
+F 0 "U7" H 1400 2450 50  0000 C CNN
+F 1 "W25Q32JVSS" H 1350 1750 50  0000 C CNN
 F 2 "Package_SO:SOIC-8_5.23x5.23mm_P1.27mm" H 1700 2100 50  0001 C CNN
 F 3 "http://www.winbond.com/resource-files/w25q32jv%20revg%2003272018%20plus.pdf" H 1700 2100 50  0001 C CNN
@@
 $EndComp
 $Comp
-L power:GND #PWR?
+L power:GND #PWR0124
 U 1 1 5F6B7D67
 P 1700 2550
-F 0 "#PWR?" H 1700 2300 50  0001 C CNN
+F 0 "#PWR0124" H 1700 2300 50  0001 C CNN
 F 1 "GND" H 1705 2377 50  0000 C CNN
 F 2 "" H 1700 2550 50  0001 C CNN
@@
 $EndComp
 $Comp
-L cerg:VCCIO #PWR?
+L cerg:VCCIO #PWR0125
 U 1 1 5F6B8568
 P 1700 1100
-F 0 "#PWR?" H 1700 950 50  0001 C CNN
+F 0 "#PWR0125" H 1700 950 50  0001 C CNN
 F 1 "VCCIO" V 1600 1100 50  0000 C CNN
 F 2 "" H 1700 1100 50  0001 C CNN
@@
 	1700 2500 1700 2550
 $Comp
-L Device:C C?
+L Device:C C16
 U 1 1 5F6B9D0D
 P 2050 1300
-F 0 "C?" H 2165 1346 50  0000 L CNN
+F 0 "C16" H 2165 1346 50  0000 L CNN
 F 1 "100n" H 2165 1255 50  0000 L CNN
 F 2 "Capacitor_SMD:C_0603_1608Metric" H 2088 1150 50  0001 C CNN
@@
 $EndComp
 $Comp
-L Device:R R?
+L Device:R R28
 U 1 1 5F6C405F
 P 2400 2000
-F 0 "R?" V 2500 1900 50  0000 C CNN
+F 0 "R28" V 2500 1900 50  0000 C CNN
 F 1 "33R" V 2500 2100 50  0000 C CNN
 F 2 "Resistor_SMD:R_0603_1608Metric" V 2330 2000 50  0001 C CNN
@@
 	2200 2000 2250 2000
 $Comp
-L Device:R R?
+L Device:R R27
 U 1 1 5F6D5097
 P 2400 1800
-F 0 "R?" V 2500 1700 50  0000 C CNN
+F 0 "R27" V 2500 1700 50  0000 C CNN
 F 1 "33R" V 2500 1900 50  0000 C CNN
 F 2 "Resistor_SMD:R_0603_1608Metric" V 2330 1800 50  0001 C CNN
@@
 	850  2000 1200 2000
 $Comp
-L Device:R R?
+L Device:R R25
 U 1 1 5F6D852C
 P 850 1450
-F 0 "R?" V 950 1350 50  0000 C CNN
+F 0 "R25" V 950 1350 50  0000 C CNN
 F 1 "4K7" V 950 1550 50  0000 C CNN
 F 2 "Resistor_SMD:R_0603_1608Metric" V 780 1450 50  0001 C CNN
@@
 Connection ~ 850  2000
 $Comp
-L cerg:VCCIO #PWR?
+L cerg:VCCIO #PWR0126
 U 1 1 5F6D9DF1
 P 850 1100
-F 0 "#PWR?" H 850 950 50  0001 C CNN
+F 0 "#PWR0126" H 850 950 50  0001 C CNN
 F 1 "VCCIO" V 750 1150 50  0000 C CNN
 F 2 "" H 850 1100 50  0001 C CNN
@@
 	2550 2000 2700 2000
 $Comp
-L power:GND #PWR?
+L power:GND #PWR0127
 U 1 1 5F777599
 P 2050 1500
-F 0 "#PWR?" H 2050 1250 50  0001 C CNN
+F 0 "#PWR0127" H 2050 1250 50  0001 C CNN
 F 1 "GND" H 2055 1327 50  0000 C CNN
 F 2 "" H 2050 1500 50  0001 C CNN
@@
 	2200 2200 2450 2200
 $Comp
-L cerg:VCCIO #PWR?
+L cerg:VCCIO #PWR0128
 U 1 1 5F79CDDC
 P 2300 2700
-F 0 "#PWR?" H 2300 2550 50  0001 C CNN
+F 0 "#PWR0128" H 2300 2550 50  0001 C CNN
 F 1 "VCCIO" H 2312 2957 50  0000 C CNN
 F 2 "" H 2300 2700 50  0001 C CNN
@@
 HOLD
 $Comp
-L Device:R R?
+L Device:R R29
 U 1 1 5F79F02C
 P 2950 750
-F 0 "R?" V 3050 650 50  0000 C CNN
+F 0 "R29" V 3050 650 50  0000 C CNN
 F 1 "1R" V 3050 850 50  0000 C CNN
 F 2 "Resistor_SMD:R_0603_1608Metric" V 2880 750 50  0001 C CNN
@@
 $EndComp
 $Comp
-L Device:R R?
+L Device:R R30
 U 1 1 5F79F615
 P 2950 1000
-F 0 "R?" V 3050 900 50  0000 C CNN
+F 0 "R30" V 3050 900 50  0000 C CNN
 F 1 "1R" V 3050 1100 50  0000 C CNN
 F 2 "Resistor_SMD:R_0603_1608Metric" V 2880 1000 50  0001 C CNN
@@
 	1150 2200 1200 2200
 $Comp
-L Device:R R?
+L Device:R R26
 U 1 1 5F7E769E
 P 1150 1750
-F 0 "R?" V 1250 1650 50  0000 C CNN
+F 0 "R26" V 1250 1650 50  0000 C CNN
 F 1 "33R" V 1250 1850 50  0000 C CNN
 F 2 "Resistor_SMD:R_0603_1608Metric" V 1080 1750 50  0001 C CNN
