File: hardware/fobos-dut/dut-artix7-a12t/target.sch (KiCad schematic (older format))
At the start: 28 parts

Commit message: artix 7 dut PCB work
Connections:
- net labels added: VCCIO
- net labels removed: +3V3
Changed lines of the file:
@@
 Wire Wire Line
 	2000 4700 2000 4900
-$Comp
-L power:+3V3 #PWR?
-U 1 1 5F2D8BB3
-P 2400 5100
-F 0 "#PWR?" H 2400 4950 50  0001 C CNN
-F 1 "+3V3" H 2415 5273 50  0000 C CNN
-F 2 "" H 2400 5100 50  0001 C CNN
-F 3 "" H 2400 5100 50  0001 C CNN
-	1    2400 5100
-	1    0    0    -1
-$EndComp
 Wire Wire Line
 	2400 5200 2400 5100
@@
 Wire Wire Line
 	3400 2850 3650 2850
+$Comp
+L cerg:VCCIO #PWR?
+U 1 1 5F26D720
+P 2400 5100
+F 0 "#PWR?" H 2400 4950 50  0001 C CNN
+F 1 "VCCIO" V 2300 5200 50  0000 C CNN
+F 2 "" H 2400 5100 50  0001 C CNN
+F 3 "" H 2400 5100 50  0001 C CNN
+	1    2400 5100
+	1    0    0    -1
+$EndComp
 $EndSCHEMATC

Commit message: artix 7 dut updates
Parts:
- gave numbers to parts that had none: 28
