File: hardware/fobos-dut/dut-artix7-a12t/power.sch (KiCad schematic (older format))
At the start: 23 parts

Commit message: artix 7 dut PCB work
Parts:
- added C?: 100nF, Capacitor_SMD:C_0603_1608Metric, symbol Device:C
- added C?: 10nF, Capacitor_SMD:C_0603_1608Metric, symbol Device:C
- added C?: 10uF, Capacitor_SMD:C_0805_2012Metric, symbol Device:C
- added Q?: FDS9435A, Package_SO:SOIC-8_3.9x4.9mm_P1.27mm, symbol Transistor_FET:FDS9435A
- added R?: 100R, Resistor_SMD:R_0603_1608Metric, symbol Device:R
- added R?: 1M, Resistor_SMD:R_0603_1608Metric, symbol Device:R
- added U?: INA225, Package_SO:MSOP-8_3x3mm_P0.65mm, symbol cerg:INA225
Connections:
- net GND: now also C?.2, R?.1
- net CW_3V3 renamed FS_3V3
- net CW_5V renamed FS_5V
- new net: C?.1, Q?.1 (S), Q?.2 (S), Q?.3 (S)
- new net: C?.2, Q?.4 (G), R?.2, R?.2
- new net: C?.1, C?.1, Q?.5 (D), Q?.6 (D), Q?.7 (D), Q?.8 (D)
- new net: C?.2, R?.1
Other:
- note added: "Soft-Start"
Changed lines of the file:
@@
 	6200 2500 6200 2650
 Text GLabel 9000 2900 2    50   Input ~ 0
-CW_3V3
+FS_3V3
 Wire Wire Line
 	1800 2150 2000 2150
@@
 	2250 1900 2150 1900
 Text GLabel 1800 2150 0    50   Input ~ 0
-CW_5V
+FS_5V
 Connection ~ 5800 1900
 $Comp
@@
 EndData
 $EndBitmap
+$Comp
+L cerg:INA225 U?
+U 1 1 5F2A6698
+P 5350 2850
+F 0 "U?" H 5350 3431 50  0000 C CNN
+F 1 "INA225" H 5350 3340 50  0000 C CNN
+F 2 "Package_SO:MSOP-8_3x3mm_P0.65mm" H 5400 2850 50  0001 C CNN
+F 3 "" H 5700 2650 50  0001 C CNN
+	1    5350 2850
+	1    0    0    -1
+$EndComp
+$Comp
+L Device:C C?
+U 1 1 5F2BA835
+P 2600 3700
+AR Path="/5F227C5D/5F2BA835" Ref="C?"  Part="1"
+AR Path="/5F449901/5F2BA835" Ref="C?"  Part="1"
+F 0 "C?" H 2715 3746 50  0000 L CNN
+F 1 "100nF" H 2715 3655 50  0000 L CNN
+F 2 "Capacitor_SMD:C_0603_1608Metric" H 2638 3550 50  0001 C CNN
+F 3 "~" H 2600 3700 50  0001 C CNN
+	1    2600 3700
+	1    0    0    -1
+$EndComp
+$Comp
+L Device:C C?
+U 1 1 5F2BAC27
+P 3900 3700
+AR Path="/5F227C5D/5F2BAC27" Ref="C?"  Part="1"
+AR Path="/5F449901/5F2BAC27" Ref="C?"  Part="1"
+F 0 "C?" H 4015 3746 50  0000 L CNN
+F 1 "10nF" H 4015 3655 50  0000 L CNN
+F 2 "Capacitor_SMD:C_0603_1608Metric" H 3938 3550 50  0001 C CNN
+F 3 "~" H 3900 3700 50  0001 C CNN
+	1    3900 3700
+	1    0    0    -1
+$EndComp
+$Comp
+L Device:R R?
+U 1 1 5F2BD9D2
+P 3400 3900
+F 0 "R?" V 3193 3900 50  0000 C CNN
+F 1 "100R" V 3284 3900 50  0000 C CNN
+F 2 "Resistor_SMD:R_0603_1608Metric" V 3330 3900 50  0001 C CNN
+F 3 "~" H 3400 3900 50  0001 C CNN
+	1    3400 3900
+	0    1    1    0
+$EndComp
+$Comp
+L Device:R R?
+U 1 1 5F2BE6B1
+P 2600 4150
+F 0 "R?" V 2393 4150 50  0000 C CNN
+F 1 "1M" V 2484 4150 50  0000 C CNN
+F 2 "Resistor_SMD:R_0603_1608Metric" V 2530 4150 50  0001 C CNN
+F 3 "~" H 2600 4150 50  0001 C CNN
+	1    2600 4150
+	-1   0    0    1
+$EndComp
+$Comp
+L Transistor_FET:FDS9435A Q?
+U 1 1 5F2C0777
+P 3100 3600
+F 0 "Q?" V 3442 3600 50  0000 C CNN
+F 1 "FDS9435A" V 3351 3600 50  0000 C CNN
+F 2 "Package_SO:SOIC-8_3.9x4.9mm_P1.27mm" H 3300 3525 50  0001 L CIN
+F 3 "https://www.onsemi.com/pub/Collateral/FDS9435A-D.PDF" V 3100 3600 50  0001 L CNN
+	1    3100 3600
+	0    1    -1   0
+$EndComp
+Wire Wire Line
+	2600 3500 2900 3500
+Wire Wire Line
+	2600 3550 2600 3500
+Wire Wire Line
+	3300 3500 3900 3500
+Wire Wire Line
+	3900 3500 3900 3550
+Wire Wire Line
+	2600 3850 2600 3900
+Wire Wire Line
+	2600 3900 3100 3900
+Wire Wire Line
+	3100 3800 3100 3900
+Connection ~ 3100 3900
+Wire Wire Line
+	3100 3900 3250 3900
+Wire Wire Line
+	3550 3900 3900 3900
+Wire Wire Line
+	3900 3900 3900 3850
+Wire Wire Line
+	2600 3900 2600 4000
+Connection ~ 2600 3900
+$Comp
+L power:GND #PWR?
+U 1 1 5F2DE57D
+P 2600 4400
+F 0 "#PWR?" H 2600 4150 50  0001 C CNN
+F 1 "GND" H 2605 4227 50  0000 C CNN
+F 2 "" H 2600 4400 50  0001 C CNN
+F 3 "" H 2600 4400 50  0001 C CNN
+	1    2600 4400
+	1    0    0    -1
+$EndComp
+Wire Wire Line
+	2600 4300 2600 4400
+$Comp
+L Device:C C?
+U 1 1 5F2E0852
+P 4350 3700
+AR Path="/5F227C5D/5F2E0852" Ref="C?"  Part="1"
+AR Path="/5F449901/5F2E0852" Ref="C?"  Part="1"
+F 0 "C?" H 4465 3746 50  0000 L CNN
+F 1 "10uF" H 4465 3655 50  0000 L CNN
+F 2 "Capacitor_SMD:C_0805_2012Metric" H 4388 3550 50  0001 C CNN
+F 3 "~" H 4350 3700 50  0001 C CNN
+	1    4350 3700
+	1    0    0    -1
+$EndComp
+Wire Wire Line
+	3900 3500 4350 3500
+Wire Wire Line
+	4350 3500 4350 3550
+Connection ~ 3900 3500
+$Comp
+L power:GND #PWR?
+U 1 1 5F2E2E50
+P 4350 4400
+F 0 "#PWR?" H 4350 4150 50  0001 C CNN
+F 1 "GND" H 4355 4227 50  0000 C CNN
+F 2 "" H 4350 4400 50  0001 C CNN
+F 3 "" H 4350 4400 50  0001 C CNN
+	1    4350 4400
+	1    0    0    -1
+$EndComp
+Wire Wire Line
+	4350 3850 4350 4400
+Text Notes 3150 3150 0    79   ~ 0
+Soft-Start
 $EndSCHEMATC

Commit message: artix 7 dut updates
Parts:
- TP1: renamed from TP?; value TestPoint -> 5V
- gave numbers to parts that had none: 29
Connections:
- net FS_5V: now also C4.1, Q1.1 (S), Q1.2 (S), Q1.3 (S); no longer JP1.1 (A)
- net +5V: now reaches C10.1, C8.1, Q1.5 (D), Q1.6 (D), Q1.7 (D), Q1.8 (D)
- net +5V: now also TP1.1
- net V_Core renamed VCC
- new net +1V0: JP1.1 (A)
Other:
- moved on the sheet: TP1

Commit message: Added LTC3633 power regulator to serve as the main system power supply
Parts:
- added C?: 10uF, symbol Device:C
- added C? (x3): 2.2uF, symbol Device:C
- added C?: 470pF, symbol Device:C
- added C?: 62pF, symbol Device:C
- added C?: 180pF, symbol Device:C
- added C?: 18pF, symbol Device:C
- added C?: 13pF, symbol Device:C
- added C? (x2): 56pF, symbol Device:C
- added C? (x5): 100nF, symbol Device:C
- added C?: 10nF, symbol Device:C
- added C? (x2): 100uF, symbol Device:C
- added C? (x2): 47uF, symbol Device:C
- added C?: 160pF, symbol Device:C
- added L?: 1.5uH, symbol Device:L
- added L?: 2.2uH, symbol Device:L
- added R?: 576KR, Resistor_SMD:R_0603_1608Metric, symbol Device:R
- added R?: 100KR, Resistor_SMD:R_0603_1608Metric, symbol Device:R
- added R?: 9.31KR, Resistor_SMD:R_0603_1608Metric, symbol Device:R
- added R?: 32.4KR, Resistor_SMD:R_0603_1608Metric, symbol Device:R
- added R? (x3): 0R, Resistor_SMD:R_0603_1608Metric, symbol Device:R
- added R? (x2): 88.7KR, Resistor_SMD:R_0603_1608Metric, symbol Device:R
- added R? (x2): 59KR, Resistor_SMD:R_0603_1608Metric, symbol Device:R
- added U?: LTC3633, symbol cerg:LTC3633
Connections:
- net labels added: INTVCC
- wire segments 85 -> 236

Commit message: Adding LTC3633 power chip to CERG lib
Parts:
- added JP?: Source, Connector_PinHeader_2.54mm:PinHeader_1x03_P2.54mm_Vertical, symbol Jumper:Jumper_3_Open
- added R?: 10KR, Resistor_SMD:R_0603_1608Metric, symbol Device:R
- added R?: 4.7KR, Resistor_SMD:R_0603_1608Metric, symbol Device:R
- gave numbers to parts that had none: 36
Connections:
- net labels added: RUN
- wire segments 236 -> 241
Other:
- moved on the sheet: C10, C4, C8, Q1, R21, R22, TP1, U5

Commit message: Removed LTC3633 dual output power switcher IC Added LTC3569 triple output power switcher IC
Parts:
- removed C17: 470pF, symbol Device:C
- removed C18: 10uF, symbol Device:C
- removed C19: 62pF, symbol Device:C
- removed C20, C22, C24: 2.2uF, symbol Device:C
- removed C21: 180pF, symbol Device:C
- removed C23: 18pF, symbol Device:C
- removed C25, C26, C27, C33, C38: 100nF, symbol Device:C
- removed C28: 10nF, symbol Device:C
- removed C29, C34: 56pF, symbol Device:C
- removed C30: 13pF, symbol Device:C
- removed C31, C36: 100uF, symbol Device:C
- removed C32, C37: 47uF, symbol Device:C
- removed C35: 160pF, symbol Device:C
- removed L3: 2.2uH, symbol Device:L
- removed L4: 1.5uH, symbol Device:L
- removed R34: 9.31KR, Resistor_SMD:R_0603_1608Metric, symbol Device:R
- removed R35: 32.4KR, Resistor_SMD:R_0603_1608Metric, symbol Device:R
- removed R36: 100KR, Resistor_SMD:R_0603_1608Metric, symbol Device:R
- removed R37: 576KR, Resistor_SMD:R_0603_1608Metric, symbol Device:R
- removed R38, R39, R40: 0R, Resistor_SMD:R_0603_1608Metric, symbol Device:R
- removed R41, R43: 59KR, Resistor_SMD:R_0603_1608Metric, symbol Device:R
- removed R42, R44: 88.7KR, Resistor_SMD:R_0603_1608Metric, symbol Device:R
- removed U8: LTC3633, symbol cerg:LTC3633
- added C? (x2): 22uF, Capacitor_SMD:C_0805_2012Metric, symbol Device:C
- added C? (x3): 20pF, Capacitor_SMD:C_0603_1608Metric, symbol Device:C
- added C? (x2): 10uF, Capacitor_SMD:C_0805_2012Metric, symbol Device:C
- added L?: 1.5uH, symbol Device:L
- added L?: 3.3uH, symbol Device:L
- added L?: 2.2uH, symbol Device:L
- added Q? (x2): MBT3904DW1, Package_TO_SOT_SMD:SOT-363_SC-70-6, symbol Transistor_BJT:MBT3904DW1
- added R?: 3.48KR, Resistor_SMD:R_0603_1608Metric, symbol Device:R
- added R? (x4): 10KR, Resistor_SMD:R_0603_1608Metric, symbol Device:R
- added R?: 0, Resistor_SMD:R_0603_1608Metric, symbol Device:R
- added R? (x3): 100KR, Resistor_SMD:R_0603_1608Metric, symbol Device:R
- added R?: 1KR, Resistor_SMD:R_0603_1608Metric, symbol Device:R
- added R? (x2): 120KR, Resistor_SMD:R_0603_1608Metric, symbol Device:R
- added R?: 57.6KR, Resistor_SMD:R_0603_1608Metric, symbol Device:R
- added U?: LTC3569EFE#PBF, symbol cerg:LTC3569EFE#PBF
Connections:
- net labels added: +1V8, +3.3V, PGOOD
- net labels removed: INTVCC
- wire segments 241 -> 181
Other:
- note added: "Add PGOOD LED"
- note added: "On-board Switching Power Supply"
- moved on the sheet: C11, C12, C13, C14, C15, J6, JP?, L2, R24, R?, U5, U6

Commit message: Finished the LTC3659 circuit - added gnd, epad to gnd net Completed PGOOD LED circuit Added slide switch to serve as ON_OFF switch
Parts:
- removed JP?: Source, Connector_PinHeader_2.54mm:PinHeader_1x03_P2.54mm_Vertical, symbol Jumper:Jumper_3_Open
- added D1: LG_L29K-G2J1-24-Z, digikey-footprints:0603, symbol dk_LED-Indication-Discrete:LG_L29K-G2J1-24-Z
- added Q3: FDV301N, digikey-footprints:SOT-23-3, symbol dk_Transistors-FETs-MOSFETs-Single:FDV301N
- added R49: 100KR, Resistor_SMD:R_0603_1608Metric, symbol Device:R
- added R50: 800R, Resistor_SMD:R_0603_1608Metric, symbol Device:R
- added S1: JS202011SCQN, digikey-footprints:Switch_Slide_JS202011SCQN, symbol dk_Slide-Switches:JS202011SCQN
- gave numbers to parts that had none: 27
Connections:
- net labels added: ON_OFF
- net labels removed: RUN
- wire segments 181 -> 197
Other:
- note removed: "Add PGOOD LED"

Commit message: Added PGOOD LED and NFET Connected INA225 to Current shunt resistor
Parts:
- added C24: 100nF, Capacitor_SMD:C_0603_1608Metric, symbol Device:C
Connections:
- net labels added: VCORE_CURRENT, VCORE_CURRENT_GAIN_0, VCORE_CURRENT_GAIN_1
- wire segments 197 -> 219
Other:
- moved on the sheet: R41, R42, R49, R50, U5
