File: hardware/fobos-dut/dut-artix7-a12t/User Button and IO.sch (KiCad schematic (older format))
At the start: 18 parts, among them Q4 FDV301N, Q5 FDV301N, Q6 FDV301N

Commit message: Preliminary placement underway Made a copy of cerg 3d model within Artix 7 dut project to resolve nagging library path issue
Parts:
- added D5: LG_L29K-G2J1-24-Z, digikey-footprints:0603, symbol dk_LED-Indication-Discrete:LG_L29K-G2J1-24-Z
- added Q7: BSS138, Package_TO_SOT_SMD:SOT-23, symbol Transistor_FET:BSS138
- added R68: 10KR, Resistor_SMD:R_0603_1608Metric, symbol Device:R
- added R69: 470R, Resistor_SMD:R_0603_1608Metric, symbol Device:R
- D2: footprint digikey-footprints:0603 -> LED_SMD:LED_0603_1608Metric
- R57, R58, R59: value 800R -> 470R
Connections:
- wire segments 47 -> 60
Other:
- note added: "User LED_4"
Changed lines of the file:
@@
 F 0 "D2" V 1947 2428 60  0000 L CNN
 F 1 "LG_L29K-G2J1-24-Z" V 2053 2428 60  0001 L CNN
-F 2 "digikey-footprints:0603" H 2250 2450 60  0001 L CNN
+F 2 "LED_SMD:LED_0603_1608Metric" H 2250 2450 60  0001 L CNN
 F 3 "https://dammedia.osram.info/media/resource/hires/osram-dam-2493945/LG%20L29K.pdf" H 2250 2550 60  0001 L CNN
 F 4 "475-2709-1-ND" H 2250 2650 60  0001 L CNN "Digi-Key_PN"
@@
 AR Path="/600CE672/600D00E4" Ref="R57"  Part="1"
 F 0 "R57" V 2250 2600 50  0000 C CNN
-F 1 "800R" V 2150 2600 50  0000 C CNN
+F 1 "470R" V 2150 2600 50  0000 C CNN
 F 2 "Resistor_SMD:R_0603_1608Metric" V 1980 2600 50  0001 C CNN
 F 3 "~" H 2050 2600 50  0001 C CNN
@@
 AR Path="/600CE672/600D0FAE" Ref="R58"  Part="1"
 F 0 "R58" V 4300 2650 50  0000 C CNN
-F 1 "800R" V 4200 2650 50  0000 C CNN
+F 1 "470R" V 4200 2650 50  0000 C CNN
 F 2 "Resistor_SMD:R_0603_1608Metric" V 4030 2650 50  0001 C CNN
 F 3 "~" H 4100 2650 50  0001 C CNN
@@
 Wire Wire Line
 	3800 2000 4100 2000
-$Comp
-L dk_Transistors-FETs-MOSFETs-Single:FDV301N Q?
-U 1 1 600D2B55
-P 5950 3100
-AR Path="/5F449901/600D2B55" Ref="Q?"  Part="1"
-AR Path="/600CE672/600D2B55" Ref="Q6"  Part="1"
-F 0 "Q6" H 6058 3153 60  0000 L CNN
-F 1 "FDV301N" H 6058 3047 60  0000 L CNN
-F 2 "digikey-footprints:SOT-23-3" H 6150 3300 60  0001 L CNN
-F 3 "https://www.onsemi.com/pub/Collateral/FDV301N-D.PDF" H 6150 3400 60  0001 L CNN
-F 4 "FDV301NCT-ND" H 6150 3500 60  0001 L CNN "Digi-Key_PN"
-F 5 "FDV301N" H 6150 3600 60  0001 L CNN "MPN"
-F 6 "Discrete Semiconductor Products" H 6150 3700 60  0001 L CNN "Category"
-F 7 "Transistors - FETs, MOSFETs - Single" H 6150 3800 60  0001 L CNN "Family"
-F 8 "https://www.onsemi.com/pub/Collateral/FDV301N-D.PDF" H 6150 3900 60  0001 L CNN "DK_Datasheet_Link"
-F 9 "/product-detail/en/on-semiconductor/FDV301N/FDV301NCT-ND/458954" H 6150 4000 60  0001 L CNN "DK_Detail_Page"
-F 10 "MOSFET N-CH 25V 220MA SOT-23" H 6150 4100 60  0001 L CNN "Description"
-F 11 "ON Semiconductor" H 6150 4200 60  0001 L CNN "Manufacturer"
-F 12 "Active" H 6150 4300 60  0001 L CNN "Status"
-	1    5950 3100
-	1    0    0    -1
-$EndComp
 $Comp
 L power:GND #PWR?
@@
 AR Path="/600CE672/600D2B76" Ref="R59"  Part="1"
 F 0 "R59" V 6150 2650 50  0000 C CNN
-F 1 "800R" V 6050 2650 50  0000 C CNN
+F 1 "470R" V 6050 2650 50  0000 C CNN
 F 2 "Resistor_SMD:R_0603_1608Metric" V 5880 2650 50  0001 C CNN
 F 3 "~" H 5950 2650 50  0001 C CNN
@@
 Text Notes 9400 2100 0    50   ~ 0
 User Button_1
+$Comp
+L dk_Transistors-FETs-MOSFETs-Single:FDV301N Q?
+U 1 1 602D02E9
+P 2050 5550
+AR Path="/5F449901/602D02E9" Ref="Q?"  Part="1"
+AR Path="/600CE672/602D02E9" Ref="Q6"  Part="1"
+F 0 "Q6" H 2158 5603 60  0000 L CNN
+F 1 "FDV301N" H 2158 5497 60  0000 L CNN
+F 2 "digikey-footprints:SOT-23-3" H 2250 5750 60  0001 L CNN
+F 3 "https://www.onsemi.com/pub/Collateral/FDV301N-D.PDF" H 2250 5850 60  0001 L CNN
+F 4 "FDV301NCT-ND" H 2250 5950 60  0001 L CNN "Digi-Key_PN"
+F 5 "FDV301N" H 2250 6050 60  0001 L CNN "MPN"
+F 6 "Discrete Semiconductor Products" H 2250 6150 60  0001 L CNN "Category"
+F 7 "Transistors - FETs, MOSFETs - Single" H 2250 6250 60  0001 L CNN "Family"
+F 8 "https://www.onsemi.com/pub/Collateral/FDV301N-D.PDF" H 2250 6350 60  0001 L CNN "DK_Datasheet_Link"
+F 9 "/product-detail/en/on-semiconductor/FDV301N/FDV301NCT-ND/458954" H 2250 6450 60  0001 L CNN "DK_Detail_Page"
+F 10 "MOSFET N-CH 25V 220MA SOT-23" H 2250 6550 60  0001 L CNN "Description"
+F 11 "ON Semiconductor" H 2250 6650 60  0001 L CNN "Manufacturer"
+F 12 "Active" H 2250 6750 60  0001 L CNN "Status"
+	1    2050 5550
+	1    0    0    -1
+$EndComp
+$Comp
+L power:GND #PWR?
+U 1 1 602D02EF
+P 2050 6300
+AR Path="/5F449901/602D02EF" Ref="#PWR?"  Part="1"
+AR Path="/600CE672/602D02EF" Ref="#PWR022"  Part="1"
+F 0 "#PWR022" H 2050 6050 50  0001 C CNN
+F 1 "GND" H 2055 6127 50  0000 C CNN
+F 2 "" H 2050 6300 50  0001 C CNN
+F 3 "" H 2050 6300 50  0001 C CNN
+	1    2050 6300
+	1    0    0    -1
+$EndComp
+$Comp
+L dk_LED-Indication-Discrete:LG_L29K-G2J1-24-Z D?
+U 1 1 602D02FE
+P 2050 4750
+AR Path="/5F449901/602D02FE" Ref="D?"  Part="1"
+AR Path="/600CE672/602D02FE" Ref="D5"  Part="1"
+F 0 "D5" V 1947 4928 60  0000 L CNN
+F 1 "LG_L29K-G2J1-24-Z" V 2053 4928 60  0001 L CNN
+F 2 "digikey-footprints:0603" H 2250 4950 60  0001 L CNN
+F 3 "https://dammedia.osram.info/media/resource/hires/osram-dam-2493945/LG%20L29K.pdf" H 2250 5050 60  0001 L CNN
+F 4 "475-2709-1-ND" H 2250 5150 60  0001 L CNN "Digi-Key_PN"
+F 5 "LG L29K-G2J1-24-Z" H 2250 5250 60  0001 L CNN "MPN"
+F 6 "Optoelectronics" H 2250 5350 60  0001 L CNN "Category"
+F 7 "LED Indication - Discrete" H 2250 5450 60  0001 L CNN "Family"
+F 8 "https://dammedia.osram.info/media/resource/hires/osram-dam-2493945/LG%20L29K.pdf" H 2250 5550 60  0001 L CNN "DK_Datasheet_Link"
+F 9 "/product-detail/en/osram-opto-semiconductors-inc/LG-L29K-G2J1-24-Z/475-2709-1-ND/1938876" H 2250 5650 60  0001 L CNN "DK_Detail_Page"
+F 10 "LED GREEN DIFFUSED 0603 SMD" H 2250 5750 60  0001 L CNN "Description"
+F 11 "OSRAM Opto Semiconductors Inc." H 2250 5850 60  0001 L CNN "Manufacturer"
+F 12 "Active" H 2250 5950 60  0001 L CNN "Status"
+	1    2050 4750
+	0    1    1    0
+$EndComp
+$Comp
+L Device:R R?
+U 1 1 602D0304
+P 2050 5100
+AR Path="/5F449901/602D0304" Ref="R?"  Part="1"
+AR Path="/600CE672/602D0304" Ref="R69"  Part="1"
+F 0 "R69" V 2250 5100 50  0000 C CNN
+F 1 "470R" V 2150 5100 50  0000 C CNN
+F 2 "Resistor_SMD:R_0603_1608Metric" V 1980 5100 50  0001 C CNN
+F 3 "~" H 2050 5100 50  0001 C CNN
+	1    2050 5100
+	1    0    0    -1
+$EndComp
+Wire Wire Line
+	2050 5350 2050 5250
+Wire Wire Line
+	2050 4950 2050 4850
+Wire Wire Line
+	1750 5650 1550 5650
+Wire Wire Line
+	1550 5650 1300 5650
+Connection ~ 1550 5650
+Wire Wire Line
+	2050 4450 2050 4550
+Text GLabel 1800 4300 2    50   Input ~ 0
+FC_3V3
+Wire Wire Line
+	1800 4300 1750 4300
+Wire Wire Line
+	1750 4300 1750 4450
+Wire Wire Line
+	1750 4450 2050 4450
+$Comp
+L Device:R R?
+U 1 1 602D0314
+P 1550 5900
+AR Path="/5F449901/602D0314" Ref="R?"  Part="1"
+AR Path="/600CE672/602D0314" Ref="R68"  Part="1"
+F 0 "R68" V 1343 5900 50  0000 C CNN
+F 1 "10KR" V 1434 5900 50  0000 C CNN
+F 2 "Resistor_SMD:R_0603_1608Metric" V 1480 5900 50  0001 C CNN
+F 3 "~" H 1550 5900 50  0001 C CNN
+	1    1550 5900
+	-1   0    0    1
+$EndComp
+Wire Wire Line
+	2050 5750 2050 6150
+Wire Wire Line
+	1550 6050 1550 6150
+Wire Wire Line
+	1550 6150 2050 6150
+Connection ~ 2050 6150
+Wire Wire Line
+	2050 6150 2050 6300
+Wire Wire Line
+	1550 5750 1550 5650
+Text Notes 1750 4150 0    50   ~ 0
+User LED_4
+$Comp
+L Transistor_FET:BSS138 Q7
+U 1 1 602D521D
+P 5850 3100
+F 0 "Q7" H 6054 3146 50  0000 L CNN
+F 1 "BSS138" H 6054 3055 50  0000 L CNN
+F 2 "Package_TO_SOT_SMD:SOT-23" H 6050 3025 50  0001 L CIN
+F 3 "https://www.fairchildsemi.com/datasheets/BS/BSS138.pdf" H 5850 3100 50  0001 L CNN
+	1    5850 3100
+	1    0    0    -1
+$EndComp
 $EndSCHEMATC

Commit message: Coarse placement of all components within board outline, began to route traces
Parts:
- removed Q4, Q5, Q6: FDV301N, digikey-footprints:SOT-23-3, symbol dk_Transistors-FETs-MOSFETs-Single:FDV301N
- added Q4, Q5, Q6: BSS138, Package_TO_SOT_SMD:SOT-23, symbol Transistor:BSS138
Connections:
- wire segments 60 -> 56
Changed lines of the file:
@@
 $EndDescr
-$Comp
-L dk_Transistors-FETs-MOSFETs-Single:FDV301N Q?
-U 1 1 600D00C3
-P 2050 3050
-AR Path="/5F449901/600D00C3" Ref="Q?"  Part="1"
-AR Path="/600CE672/600D00C3" Ref="Q4"  Part="1"
-F 0 "Q4" H 2158 3103 60  0000 L CNN
-F 1 "FDV301N" H 2158 2997 60  0000 L CNN
-F 2 "digikey-footprints:SOT-23-3" H 2250 3250 60  0001 L CNN
-F 3 "https://www.onsemi.com/pub/Collateral/FDV301N-D.PDF" H 2250 3350 60  0001 L CNN
-F 4 "FDV301NCT-ND" H 2250 3450 60  0001 L CNN "Digi-Key_PN"
-F 5 "FDV301N" H 2250 3550 60  0001 L CNN "MPN"
-F 6 "Discrete Semiconductor Products" H 2250 3650 60  0001 L CNN "Category"
-F 7 "Transistors - FETs, MOSFETs - Single" H 2250 3750 60  0001 L CNN "Family"
-F 8 "https://www.onsemi.com/pub/Collateral/FDV301N-D.PDF" H 2250 3850 60  0001 L CNN "DK_Datasheet_Link"
-F 9 "/product-detail/en/on-semiconductor/FDV301N/FDV301NCT-ND/458954" H 2250 3950 60  0001 L CNN "DK_Detail_Page"
-F 10 "MOSFET N-CH 25V 220MA SOT-23" H 2250 4050 60  0001 L CNN "Description"
-F 11 "ON Semiconductor" H 2250 4150 60  0001 L CNN "Manufacturer"
-F 12 "Active" H 2250 4250 60  0001 L CNN "Status"
-	1    2050 3050
-	1    0    0    -1
-$EndComp
 $Comp
 L power:GND #PWR?
@@
 	2050 2450 2050 2350
 Wire Wire Line
-	1750 3150 1550 3150
-Wire Wire Line
-	1550 3150 1300 3150
-Connection ~ 1550 3150
-Wire Wire Line
 	2050 1950 2050 2050
 Text GLabel 1800 1800 2    50   Input ~ 0
@@
 Wire Wire Line
 	1750 1950 2050 1950
-$Comp
-L dk_Transistors-FETs-MOSFETs-Single:FDV301N Q?
-U 1 1 600D0F8D
-P 4100 3100
-AR Path="/5F449901/600D0F8D" Ref="Q?"  Part="1"
-AR Path="/600CE672/600D0F8D" Ref="Q5"  Part="1"
-F 0 "Q5" H 4208 3153 60  0000 L CNN
-F 1 "FDV301N" H 4208 3047 60  0000 L CNN
-F 2 "digikey-footprints:SOT-23-3" H 4300 3300 60  0001 L CNN
-F 3 "https://www.onsemi.com/pub/Collateral/FDV301N-D.PDF" H 4300 3400 60  0001 L CNN
-F 4 "FDV301NCT-ND" H 4300 3500 60  0001 L CNN "Digi-Key_PN"
-F 5 "FDV301N" H 4300 3600 60  0001 L CNN "MPN"
-F 6 "Discrete Semiconductor Products" H 4300 3700 60  0001 L CNN "Category"
-F 7 "Transistors - FETs, MOSFETs - Single" H 4300 3800 60  0001 L CNN "Family"
-F 8 "https://www.onsemi.com/pub/Collateral/FDV301N-D.PDF" H 4300 3900 60  0001 L CNN "DK_Datasheet_Link"
-F 9 "/product-detail/en/on-semiconductor/FDV301N/FDV301NCT-ND/458954" H 4300 4000 60  0001 L CNN "DK_Detail_Page"
-F 10 "MOSFET N-CH 25V 220MA SOT-23" H 4300 4100 60  0001 L CNN "Description"
-F 11 "ON Semiconductor" H 4300 4200 60  0001 L CNN "Manufacturer"
-F 12 "Active" H 4300 4300 60  0001 L CNN "Status"
-	1    4100 3100
-	1    0    0    -1
-$EndComp
 $Comp
 L power:GND #PWR?
@@
 	4100 2500 4100 2400
 Wire Wire Line
-	3800 3200 3600 3200
-Wire Wire Line
-	3600 3200 3350 3200
-Connection ~ 3600 3200
-Wire Wire Line
 	4100 2000 4100 2100
 Text GLabel 3850 1850 2    50   Input ~ 0
@@
 	5950 2500 5950 2400
 Wire Wire Line
-	5650 3200 5450 3200
-Wire Wire Line
-	5450 3200 5200 3200
-Connection ~ 5450 3200
-Wire Wire Line
 	5950 2000 5950 2100
 Text GLabel 5700 1850 2    50   Input ~ 0
@@
 	5950 3700 5950 3850
 Wire Wire Line
-	5450 3300 5450 3200
-Wire Wire Line
-	3600 3300 3600 3200
-Wire Wire Line
 	3600 3600 3600 3700
 Wire Wire Line
@@
 Wire Wire Line
 	4100 3700 4100 3850
-Wire Wire Line
-	1550 3150 1550 3250
 Wire Wire Line
 	1550 3550 1550 3650
@@
 Text Notes 9400 2100 0    50   ~ 0
 User Button_1
-$Comp
-L dk_Transistors-FETs-MOSFETs-Single:FDV301N Q?
-U 1 1 602D02E9
-P 2050 5550
-AR Path="/5F449901/602D02E9" Ref="Q?"  Part="1"
-AR Path="/600CE672/602D02E9" Ref="Q6"  Part="1"
-F 0 "Q6" H 2158 5603 60  0000 L CNN
-F 1 "FDV301N" H 2158 5497 60  0000 L CNN
-F 2 "digikey-footprints:SOT-23-3" H 2250 5750 60  0001 L CNN
-F 3 "https://www.onsemi.com/pub/Collateral/FDV301N-D.PDF" H 2250 5850 60  0001 L CNN
-F 4 "FDV301NCT-ND" H 2250 5950 60  0001 L CNN "Digi-Key_PN"
-F 5 "FDV301N" H 2250 6050 60  0001 L CNN "MPN"
-F 6 "Discrete Semiconductor Products" H 2250 6150 60  0001 L CNN "Category"
-F 7 "Transistors - FETs, MOSFETs - Single" H 2250 6250 60  0001 L CNN "Family"
-F 8 "https://www.onsemi.com/pub/Collateral/FDV301N-D.PDF" H 2250 6350 60  0001 L CNN "DK_Datasheet_Link"
-F 9 "/product-detail/en/on-semiconductor/FDV301N/FDV301NCT-ND/458954" H 2250 6450 60  0001 L CNN "DK_Detail_Page"
-F 10 "MOSFET N-CH 25V 220MA SOT-23" H 2250 6550 60  0001 L CNN "Description"
-F 11 "ON Semiconductor" H 2250 6650 60  0001 L CNN "Manufacturer"
-F 12 "Active" H 2250 6750 60  0001 L CNN "Status"
-	1    2050 5550
-	1    0    0    -1
-$EndComp
 $Comp
 L power:GND #PWR?
@@
 	2050 4950 2050 4850
 Wire Wire Line
-	1750 5650 1550 5650
-Wire Wire Line
-	1550 5650 1300 5650
-Connection ~ 1550 5650
-Wire Wire Line
 	2050 4450 2050 4550
 Text GLabel 1800 4300 2    50   Input ~ 0
@@
 Wire Wire Line
 	2050 6150 2050 6300
-Wire Wire Line
-	1550 5750 1550 5650
 Text Notes 1750 4150 0    50   ~ 0
 User LED_4
@@
 	1    0    0    -1
 $EndComp
+$Comp
+L Transistor:BSS138 Q5
+U 1 1 605337F1
+P 4000 3100
+F 0 "Q5" H 4204 3146 50  0000 L CNN
+F 1 "BSS138" H 4204 3055 50  0000 L CNN
+F 2 "Package_TO_SOT_SMD:SOT-23" H 4200 3025 50  0001 L CIN
+F 3 "https://www.onsemi.com/pub/Collateral/BSS138-D.PDF" H 4000 3100 50  0001 L CNN
+	1    4000 3100
+	1    0    0    -1
+$EndComp
+$Comp
+L Transistor:BSS138 Q4
+U 1 1 60535EA9
+P 1950 3050
+F 0 "Q4" H 2154 3096 50  0000 L CNN
+F 1 "BSS138" H 2154 3005 50  0000 L CNN
+F 2 "Package_TO_SOT_SMD:SOT-23" H 2150 2975 50  0001 L CIN
+F 3 "https://www.onsemi.com/pub/Collateral/BSS138-D.PDF" H 1950 3050 50  0001 L CNN
+	1    1950 3050
+	1    0    0    -1
+$EndComp
+$Comp
+L Transistor:BSS138 Q6
+U 1 1 60537AA7
+P 1950 5550
+F 0 "Q6" H 2154 5596 50  0000 L CNN
+F 1 "BSS138" H 2154 5505 50  0000 L CNN
+F 2 "Package_TO_SOT_SMD:SOT-23" H 2150 5475 50  0001 L CIN
+F 3 "https://www.onsemi.com/pub/Collateral/BSS138-D.PDF" H 1950 5550 50  0001 L CNN
+	1    1950 5550
+	1    0    0    -1
+$EndComp
+Wire Wire Line
+	1750 5550 1550 5550
+Wire Wire Line
+	1550 5550 1550 5750
+Wire Wire Line
+	1750 3050 1550 3050
+Wire Wire Line
+	1550 3050 1550 3250
+Wire Wire Line
+	3800 3100 3600 3100
+Wire Wire Line
+	3600 3100 3600 3300
+Wire Wire Line
+	5650 3100 5450 3100
+Wire Wire Line
+	5450 3100 5450 3300
 $EndSCHEMATC

Commit message: ARTIX 7 DUT Layout is 80% done
Connections:
- net labels added: USER_BTN_1, USER_BTN_2, USER_LED_1, USER_LED_2, USER_LED_3, USER_LED_4
- wire segments 56 -> 62
Other:
- note added: "User Button_2"
- note added: "User LED_1"
- note added: "User LED_2\n"
- note added: "User LED_3"
- note removed: "User Button_0"
- note removed: "User LED_0"
- note removed: "User LED_1\n"
- note removed: "User LED_2"
Changed lines of the file:
@@
 	5650 2000 5950 2000
 Text Notes 7200 2100 0    50   ~ 0
-User Button_0
+User Button_1
 $Comp
 L Device:R R?
@@
 	2050 3650 2050 3800
 Text Notes 1700 1650 0    50   ~ 0
-User LED_0
+User LED_1
 Text Notes 3800 1700 0    50   ~ 0
-User LED_1\n
+User LED_2\n
 Text Notes 5650 1700 0    50   ~ 0
-User LED_2
+User LED_3
 $Comp
 L dk_Tactile-Switches:1825910-6 S4
@@
 	7150 2700 7350 2700
 Text Notes 9400 2100 0    50   ~ 0
-User Button_1
+User Button_2
 $Comp
 L power:GND #PWR?
@@
 Wire Wire Line
 	5450 3100 5450 3300
+Text GLabel 1300 5550 0    50   Input ~ 0
+USER_LED_4
+Wire Wire Line
+	1550 5550 1300 5550
+Connection ~ 1550 5550
+Text GLabel 5200 3100 0    50   Input ~ 0
+USER_LED_3
+Wire Wire Line
+	5450 3100 5200 3100
+Text GLabel 3350 3100 0    50   Input ~ 0
+USER_LED_2
+Wire Wire Line
+	3600 3100 3350 3100
+Text GLabel 1300 3050 0    50   Input ~ 0
+USER_LED_1
+Wire Wire Line
+	1550 3050 1300 3050
+Text GLabel 10550 2700 2    50   Input ~ 0
+USER_BTN_2
+Text GLabel 8450 2700 2    50   Input ~ 0
+USER_BTN_1
+Wire Wire Line
+	8450 2700 8250 2700
+Wire Wire Line
+	10550 2700 10400 2700
 $EndSCHEMATC

Commit message: Added Manufacturer Part Number, Manufacturer to all components except ferrite beads Added digikey quote
Parts:
- removed S4, S5: 1825910-6, digikey-footprints:Switch_Tactile_THT_6x6mm, symbol dk_Tactile-Switches:1825910-6
- added S4, S5: 1825910-6, cerg:Switch_Tactile_THT_6x6mm, symbol cerg:1825910-6
- D3, D4, D5: footprint digikey-footprints:0603 -> LED_SMD:LED_0603_1608Metric
- Q4, Q5, Q6, Q7: Description (none) -> MOSFET N-CH 50V 220MA SOT23-3; MPN (none) -> BSS138; Manufacturer (none) -> ON Semiconductor
- R57, R58, R59, R69: Description (none) -> RES 470 OHM 5% 1/10W 0603 SMD; MPN (none) -> ERJ-U03J471V; Manufacturer (none) -> Panasonic Electronic Components
- R60, R61, R62, R63, R64, R65, R66, R68: Description (none) -> RES SMD 10K OHM 1% 1/10W 0603; MPN (none) -> ERJ-3EKF1002V; Manufacturer (none) -> Panasonic Electronic Components
