File: hardware/fobos-shield/fobosshield.kicad_pcb (KiCad board)
At the start: 4 copper layers, 76.2 x 71.1 mm, 170 parts, among them J1 Target, J10 ADCin, J11 PP1, J12 PP2, J13 Clock, J14 Trigger, J15 CSM5VCur, J16 Conn_01x01, J17 Barrel_Jack_Switch, J18 Conn_01x02, J19 Conn_01x02, J2 Glitch, J20 CSM3V3Cur, J21 GND, J22 GND, J23 CSM5VCur, J24 Conn_01x02, J25 V_Var, J26 AUX, J27 GNDP, J3 Analog, J4 IOH, J5 SPI, J6 Analog2, J7 Power, J8 IOL, J9 SPI2, Q1 IRF7807Z, Q2 IRLML2502, Q3 BSS138L, U1 RB-0509D, U10 INA225, U11 INA225, U12 LD1117S33TR_SOT223, U13 INA225, U2 REE-0505S, U3 LM317L_SO8, U4 LM337L_SO8, U5 LD59015, U6 LP3985IM5-3.0, U7 AD8331, U8 TPS7A7100_VQFN20, U9 AD9215

Commit message: FOBOS Shield rev2 ready for review
Parts:
- C47, C48, C49, L5: moved to F.Cu
- moved R5 22.4 mm to (89.7, 81.0)
- moved U3 21.8 mm to (96.9, 82.9)
- moved C1 21.8 mm to (92.2, 85.6)
- moved C4 21.4 mm to (103.9, 82.0)
- moved R7 20.9 mm to (92.2, 81.8)
- moved R18 15.2 mm to (88.6, 49.5)
- moved D3 15.2 mm to (107.2, 83.9), turned to 180 degrees
- moved C3 15.2 mm to (94.0, 87.4), turned to 90 degrees
- moved R26 15.2 mm to (110.5, 83.6)
- moved L5 15.0 mm to (89.9, 45.2)
- moved C47 15.0 mm to (87.5, 44.4)
- moved C48 15.0 mm to (89.9, 43.7)
- moved C49 15.0 mm to (89.9, 42.2)
- moved C6 14.9 mm to (99.8, 87.4)
- moved REF** 14.7 mm to (41.1, 91.2)
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Routing:
- net /Power/GNDP: track 0.00 -> 137.7 mm, vias 0 -> 5
- net /Power/+7V8P: track 0.00 -> 42.9 mm, vias 0 -> 1
- net /Power/-7V8P: track 0.00 -> 42.6 mm, vias 0 -> 2
- net /Power/3V3P: track 0.00 -> 27.1 mm
- net Net-(J11-Pad3): track 0.00 -> 23.7 mm
- net Net-(C2-Pad2): track 0.00 -> 23.4 mm, vias 0 -> 1
- net Net-(C3-Pad1): track 0.00 -> 12.2 mm, vias 0 -> 1
- net Net-(C1-Pad1): track 0.00 -> 12.0 mm, vias 0 -> 1
- net VCC5V0: track 94.3 -> 102.0 mm
- net Net-(C52-Pad1): track 18.5 -> 23.9 mm
- net VCC3V3: track 84.5 -> 79.9 mm
- net Net-(R23-Pad2): track 0.00 -> 4.27 mm
- net Net-(D4-Pad2): track 0.00 -> 4.01 mm, vias 0 -> 1
- net Net-(D6-Pad2): track 0.00 -> 3.94 mm, vias 0 -> 1
- net Net-(D2-Pad2): track 0.00 -> 3.84 mm, vias 0 -> 1
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- added copper zone on F.Cu, net /Power/GNDP
Other:
- board text removed: "3V3"

Commit message: touchups on FOBOS Shield PCB
Routing:
- net /Power/GNDP: vias 5 -> 20

Commit message: starting to fill areas
Routing:
- net 5Vclean: track 17.4 -> 12.7 mm, vias 0 -> 4
- net FC_3V3: track 121.4 -> 118.8 mm
- net FC_5V: track 147.2 -> 146.2 mm
- net CSM5VCur: track 58.9 -> 58.1 mm
- net CSM5VGain1: track 54.8 -> 54.1 mm
- net CSM5VGain0: track 56.6 -> 56.0 mm
- added copper zone on In2.Cu, net /Power/GNDP
- added copper zone on F.Cu, net 5Vclean
- added copper zone on In2.Cu, net 5Vclean
- added copper zone on B.Cu, net GNDA
