File: hardware/fobos-dut/dut-artix7-a12t-cpg238/fpgapower.kicad_sch (KiCad schematic)
At the start: 13 parts

Commit message: transitioned artix-7 dut to Kikad 6
Parts:
- C38: renamed from C?; value (none) -> 100uF; footprint (none) -> Capacitor_SMD:C_1210_3225Metric_Pad1.33x2.70mm_HandSolder
- C39, C47, C55: renamed from C?; value (none) -> 47uF; footprint (none) -> Capacitor_SMD:C_0603_1608Metric_Pad1.08x0.95mm_HandSolder
- C40, C41: renamed from C?; value (none) -> 4.7uF; footprint (none) -> Capacitor_SMD:C_0402_1005Metric_Pad0.74x0.62mm_HandSolder
- C42, C43, C44, C45, C46, C56: renamed from C?; value (none) -> .47uF; footprint (none) -> Capacitor_SMD:C_0402_1005Metric_Pad0.74x0.62mm_HandSolder
- U1: renamed from U?; value (none) -> XC7A12T-CPG238; footprint (none) -> Package_BGA:Xilinx_CPG238
