File: hardware/fobos-dut/dut-artix7-a12t-cpg238/power.kicad_sch (KiCad schematic)
At the start: 76 parts

Commit message: transitioned artix-7 dut to Kikad 6
Parts:
- removed TP6, TP7, TP8, TP9: (no value), symbol cerg:5281
- added JP?: Shunt1V8, Connector_PinHeader_2.54mm:PinHeader_1x02_P2.54mm_Vertical, symbol Jumper:Jumper_2_Open
- added JP?: Shunt3V3, Connector_PinHeader_2.54mm:PinHeader_1x02_P2.54mm_Vertical, symbol Jumper:Jumper_2_Open
- C10, C22, C23, C6: renamed from C?; value (none) -> 10uF; footprint (none) -> Capacitor_SMD:C_0805_2012Metric
- C11, C13, C14, C24, C4, C5: renamed from C?; value (none) -> 100nF; footprint (none) -> Capacitor_SMD:C_0603_1608Metric
- C12: renamed from C?; value (none) -> 4n7; footprint (none) -> Capacitor_SMD:C_0603_1608Metric
- C15: renamed from C?; value (none) -> 2u2; footprint (none) -> Capacitor_SMD:C_0805_2012Metric
- C17, C21: renamed from C?; value (none) -> 22uF; footprint (none) -> Capacitor_SMD:C_0805_2012Metric
- C18, C19, C20: renamed from C?; value (none) -> 20pF; footprint (none) -> Capacitor_SMD:C_0603_1608Metric
- C7: value (none) -> 47uF6.3V; footprint (none) -> Capacitor_SMD:C_0805_2012Metric
- C8: renamed from C?; value (none) -> 10nF; footprint (none) -> Capacitor_SMD:C_0603_1608Metric
- C9: value (none) -> 100nF; footprint (none) -> Capacitor_SMD:C_0603_1608Metric
- D1: value (none) -> LG_L29K-G2J1-24-Z; footprint (none) -> LED_SMD:LED_0603_1608Metric
- F1: value (none) -> MF-MSMF050-2; footprint (none) -> Fuse:Fuse_1206_3216Metric
- J3, J8: value (none) -> 575-8; footprint (none) -> cerg:575-8
- J4: renamed from J?; value (none) -> Glitch; footprint (none) -> cerg:SMA-JOHNSON-142-0701-201
- J5: value (none) -> Conn_01x02; footprint (none) -> Connector_Molex:Molex_KK-254_AE-6410-02A_1x02_P2.54mm_Vertical
- J6, J9: renamed from J?; value (none) -> Measure; footprint (none) -> cerg:SMA-JOHNSON-142-0701-801
- JP1: value (none) -> Source; footprint (none) -> Connector_PinHeader_2.54mm:PinHeader_1x03_P2.54mm_Vertical
- JP2: value (none) -> CurProbe; footprint (none) -> Connector_PinHeader_2.54mm:PinHeader_1x02_P2.54mm_Vertical
- JP3: renamed from JP?; value (none) -> Shunt1V; footprint (none) -> Connector_PinHeader_2.54mm:PinHeader_1x02_P2.54mm_Vertical
- L1, L2: value (none) -> 1k/500mA; footprint (none) -> Inductor_SMD:L_0603_1608Metric
- L3: value (none) -> 1.5uH; footprint (none) -> cerg:L_SRN2012
- L4: value (none) -> 3.3uH; footprint (none) -> cerg:L_BRC2012
- L5: value (none) -> 2.2uH; footprint (none) -> cerg:L_SRN2012
- Q1: value (none) -> FDS9435A; footprint (none) -> Package_SO:SOIC-8_3.9x4.9mm_P1.27mm
- Q2, Q8: value (none) -> MMBT3904; footprint (none) -> Package_TO_SOT_SMD:SOT-23
- Q3: value (none) -> BSS138; footprint (none) -> Package_TO_SOT_SMD:SOT-23
- R21: value (none) -> 1M; footprint (none) -> Resistor_SMD:R_0603_1608Metric
- R22: value (none) -> 100R; footprint (none) -> Resistor_SMD:R_0603_1608Metric
- R23: renamed from R?; value (none) -> 0R1; footprint (none) -> Resistor_SMD:R_1206_3216Metric
- R24: value (none) -> 49R9; footprint (none) -> Resistor_SMD:R_0603_1608Metric
- R34: value (none) -> 3.48KR; footprint (none) -> Resistor_SMD:R_0603_1608Metric
- R35, R42, R70, R71: value (none) -> 10KR; footprint (none) -> Resistor_SMD:R_0603_1608Metric
- R36: value (none) -> 1KR; footprint (none) -> Resistor_SMD:R_0603_1608Metric
- R37: value (none) -> 0R; footprint (none) -> Resistor_SMD:R_0603_1608Metric
- R38, R39, R40, R49: value (none) -> 100KR; footprint (none) -> Resistor_SMD:R_0603_1608Metric
- R41: value (none) -> 4.7KR; footprint (none) -> Resistor_SMD:R_0603_1608Metric
- R43: value (none) -> 30K; footprint (none) -> Resistor_SMD:R_0603_1608Metric
- R44: value (none) -> 150K; footprint (none) -> Resistor_SMD:R_0603_1608Metric
- R45: value (none) -> 180K; footprint (none) -> Resistor_SMD:R_0603_1608Metric
- R46, R47: value (none) -> 120KR; footprint (none) -> Resistor_SMD:R_0603_1608Metric
- R48: value (none) -> 57.6KR; footprint (none) -> Resistor_SMD:R_0603_1608Metric
- R50: value (none) -> 800R; footprint (none) -> Resistor_SMD:R_0603_1608Metric
- R75, R76: value (none) -> 0R1; footprint (none) -> Resistor_SMD:R_1206_3216Metric
- S1: value (none) -> JS202011SCQN; footprint (none) -> cerg:Switch_Slide_JS202011SCQN
- SW2: value (none) -> SW_DIP_x03; footprint (none) -> cerg:DS04-254-2-03BK-SMT
- TP1, TP5: value (none) -> 5281; footprint (none) -> cerg:5281
- U5: value (none) -> INA225; footprint (none) -> Package_SO:MSOP-8_3x3mm_P0.65mm
- U6: value (none) -> BGA2801; footprint (none) -> Package_TO_SOT_SMD:SOT-363_SC-70-6
- U8: value (none) -> LTC3569EFE#PBF; footprint (none) -> cerg:TSSOP-16-1EP_W4.40mm
Connections:
- net +1V8: now also JP?.2 (B); no longer R34.2
- net +3V3: now also JP?.2 (B)
- net +5V: now also C24.1, U5.3 (Vs)
- net FC_3V3: no longer C24.1, U5.3 (Vs)
- net pre1V8: now also R34.2, JP?.1 (A)
- net pre3V3: now also JP?.1 (A)
Other:
- moved on the sheet: C11, J4, R24, R75, R76
